File: First.sch (KiCad schematic (older format))
At the start: 42 parts, among them P1 BNC, T1 TRANSFO2CT

Commit message: Annotate parts
Parts:
- gave numbers to parts that had none: 29
- renumbered C1 to C2, C2 to C4, D1 to D3, R3 to R4, R4 to R5
Connections:
- net at T3.4 (SB): now also SP2.1
- no-connect marks 0 -> 2
Other:
- moved on the sheet: C1, C2, C3, C4, C5, C6, C7, D1, D2, D3, D4, L1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
